File: teensy3.2/teensy3.2.sch (KiCad schematic (older format))
At the start: 33 parts, among them J1 USB_B_Micro, J2 Conn_01x26, J3 Conn_01x26, SW1 Prog, U1 LP38691SD-3.3, U2 MKL02Z32VFG4, U3 MK20DX256VLH7, Y1 32.768 KHz, Y2 16 MHz

Commit message: ajustes revision pcb
Connections:
- net AGND renamed GNDA
Changed lines of the file:
@@
 Wire Wire Line
 	2150 3650 2150 3700
-Wire Wire Line
-	2150 3700 2050 3700
-Wire Wire Line
-	2150 4000 2050 4000
 Connection ~ 1400 3250
 Wire Wire Line
@@
 Wire Wire Line
 	2150 3700 2150 3750
-Connection ~ 2150 4000
 Wire Wire Line
 	2150 3950 2150 4000
@@
 Wire Wire Line
 	8900 6200 8850 6200
-Text Label 2050 4000 2    50   ~ 0
-AGND
-Text Label 8850 6000 2    50   ~ 0
-AGND
-Text Label 2050 3700 2    50   ~ 0
+Text Label 3250 3700 2    50   ~ 0
 AREF
 Text Label 8850 5900 2    50   ~ 0
@@
 Wire Wire Line
 	8900 5300 8850 5300
-Wire Wire Line
-	8900 6000 8850 6000
 $Comp
 L Connector_Generic:Conn_01x26 J2
@@
 L power:+3.3V #PWR0105
 U 1 1 5F150E49
-P 8450 6100
-F 0 "#PWR0105" H 8450 5950 50  0001 C CNN
-F 1 "+3.3V" H 8465 6273 50  0000 C CNN
-F 2 "" H 8450 6100 50  0001 C CNN
-F 3 "" H 8450 6100 50  0001 C CNN
-	1    8450 6100
+P 8400 5950
+F 0 "#PWR0105" H 8400 5800 50  0001 C CNN
+F 1 "+3.3V" H 8415 6123 50  0000 C CNN
+F 2 "" H 8400 5950 50  0001 C CNN
+F 3 "" H 8400 5950 50  0001 C CNN
+	1    8400 5950
 	1    0    0    -1
 $EndComp
@@
 Wire Wire Line
 	6150 5900 8000 5900
-Wire Wire Line
-	8900 6100 8450 6100
 Wire Wire Line
 	7300 3400 7300 4550
@@
 Wire Wire Line
 	8150 5200 8900 5200
+$Comp
+L power:GNDA #PWR?
+U 1 1 5EE79EA4
+P 2650 4050
+F 0 "#PWR?" H 2650 3800 50  0001 C CNN
+F 1 "GNDA" H 2655 3877 50  0000 C CNN
+F 2 "" H 2650 4050 50  0001 C CNN
+F 3 "" H 2650 4050 50  0001 C CNN
+	1    2650 4050
+	1    0    0    -1
+$EndComp
+Wire Wire Line
+	2650 4050 2650 4000
+$Comp
+L power:GNDA #PWR?
+U 1 1 5EE8C512
+P 8550 6200
+F 0 "#PWR?" H 8550 5950 50  0001 C CNN
+F 1 "GNDA" H 8555 6027 50  0000 C CNN
+F 2 "" H 8550 6200 50  0001 C CNN
+F 3 "" H 8550 6200 50  0001 C CNN
+	1    8550 6200
+	1    0    0    -1
+$EndComp
+Wire Wire Line
+	8550 6000 8550 6200
+Wire Wire Line
+	8550 6000 8900 6000
+Wire Wire Line
+	8400 6100 8400 5950
+Wire Wire Line
+	8400 6100 8900 6100
 $EndSCHEMATC

Commit message: ajustes para revision final
Parts:
- C1, C10, C11, C5, C6, C7, C8: symbol Device:CP_Small -> Device:C_Small
Connections:
- net LED: no longer names the net of D2.2 (A), J2.25 (Pin_25), U3.50 (PTC5)
Other:
- moved on the sheet: D2, R4
Changed lines of the file:
@@
 	2150 1450 2250 1450
 $Comp
-L Device:CP_Small C1
+L Device:C_Small C1
 U 1 1 5ED2F4B0
 P 6100 1700
@@
 	6150 3000 6300 3000
 $Comp
-L Device:CP_Small C5
+L Device:C_Small C5
 U 1 1 5EDEA1B1
 P 1050 5550
@@
 	3950 3100 3950 3050
 $Comp
-L Device:CP_Small C6
+L Device:C_Small C6
 U 1 1 5EE02822
 P 3950 2900
@@
 $EndComp
 $Comp
-L Device:CP_Small C7
+L Device:C_Small C7
 U 1 1 5EE05B6C
 P 4350 2900
@@
 $EndComp
 $Comp
-L Device:CP_Small C8
+L Device:C_Small C8
 U 1 1 5EE08BA9
 P 4750 2900
@@
 	3950 3050 3950 3000
 $Comp
-L Device:CP_Small C11
+L Device:C_Small C11
 U 1 1 5EEA4DB3
 P 4750 4050
@@
 Wire Wire Line
 	2150 3950 2150 4000
-$Comp
-L Device:CP_Small C10
-U 1 1 5EEBAC56
-P 2150 3850
-F 0 "C10" H 2238 3896 50  0000 L CNN
-F 1 "0.1uF" H 2238 3805 50  0000 L CNN
-F 2 "Capacitor_SMD:C_0805_2012Metric" H 2150 3850 50  0001 C CNN
-F 3 "~" H 2150 3850 50  0001 C CNN
-	1    2150 3850
-	1    0    0    -1
-$EndComp
 Wire Wire Line
 	3950 3050 4350 3050
@@
 Wire Wire Line
 	8750 800  8750 1000
-Text Notes 9300 3600 0    50   ~ 10
+Text Notes 9700 3650 0    50   ~ 10
 Pin\nHeaders
 Wire Wire Line
-	10250 4150 10250 4100
+	9350 4050 9350 4000
 $Comp
 L power:GND #PWR019
 U 1 1 5EDAE460
-P 10250 4500
-F 0 "#PWR019" H 10250 4250 50  0001 C CNN
-F 1 "GND" H 10255 4327 50  0000 C CNN
-F 2 "" H 10250 4500 50  0001 C CNN
-F 3 "" H 10250 4500 50  0001 C CNN
-	1    10250 4500
+P 9350 4400
+F 0 "#PWR019" H 9350 4150 50  0001 C CNN
+F 1 "GND" H 9355 4227 50  0000 C CNN
+F 2 "" H 9350 4400 50  0001 C CNN
+F 3 "" H 9350 4400 50  0001 C CNN
+	1    9350 4400
 	1    0    0    -1
 $EndComp
@@
 L Device:R R4
 U 1 1 5EDADF39
-P 10250 4300
-F 0 "R4" H 10050 4400 50  0000 L CNN
-F 1 "470" H 10000 4300 50  0000 L CNN
-F 2 "Resistor_SMD:R_0805_2012Metric" V 10180 4300 50  0001 C CNN
-F 3 "~" H 10250 4300 50  0001 C CNN
-	1    10250 4300
+P 9350 4200
+F 0 "R4" H 9450 4250 50  0000 L CNN
+F 1 "470" H 9450 4150 50  0000 L CNN
+F 2 "Resistor_SMD:R_0805_2012Metric" V 9280 4200 50  0001 C CNN
+F 3 "~" H 9350 4200 50  0001 C CNN
+	1    9350 4200
 	1    0    0    -1
 $EndComp
@@
 L Device:LED D2
 U 1 1 5EDAC907
-P 10250 3950
-F 0 "D2" V 10300 4150 50  0000 R CNN
-F 1 "LED" V 10200 4150 50  0000 R CNN
-F 2 "LED_SMD:LED_0805_2012Metric" H 10250 3950 50  0001 C CNN
-F 3 "~" H 10250 3950 50  0001 C CNN
-	1    10250 3950
+P 9350 3850
+F 0 "D2" V 9400 3750 50  0000 R CNN
+F 1 "LED" V 9300 3750 50  0000 R CNN
+F 2 "LED_SMD:LED_0805_2012Metric" H 9350 3850 50  0001 C CNN
+F 3 "~" H 9350 3850 50  0001 C CNN
+	1    9350 3850
 	0    -1   -1   0
 $EndComp
@@
 $EndComp
 Wire Wire Line
-	10250 4500 10250 4450
+	9350 4400 9350 4350
 Wire Wire Line
 	6150 6200 8150 6200
@@
 Text Label 8850 1900 2    50   ~ 0
 J2_11
-Text Label 10250 3800 0    50   ~ 0
-LED
-Text Label 8750 3800 0    50   ~ 0
-LED
 $Comp
 L Mechanical:Fiducial FID2
@@
 	7450 4750 7450 3800
 Wire Wire Line
-	7450 3800 8900 3800
+	7450 3800 8800 3800
 Wire Wire Line
 	6150 4750 7450 4750
@@
 Wire Wire Line
 	8400 6100 8900 6100
+Wire Wire Line
+	9350 3700 9350 3550
+Wire Wire Line
+	9350 3550 8800 3550
+Wire Wire Line
+	8800 3550 8800 3800
+Connection ~ 8800 3800
+Wire Wire Line
+	8800 3800 8900 3800
+$Comp
+L Device:C_Small C10
+U 1 1 5EEBAC56
+P 2150 3850
+F 0 "C10" H 2238 3896 50  0000 L CNN
+F 1 "0.1uF" H 2238 3805 50  0000 L CNN
+F 2 "Capacitor_SMD:C_0805_2012Metric" H 2150 3850 50  0001 C CNN
+F 3 "~" H 2150 3850 50  0001 C CNN
+	1    2150 3850
+	1    0    0    -1
+$EndComp
 $EndSCHEMATC
