File: teensy3.2/teensy3.2.kicad_pcb (KiCad board)
At the start: 2 copper layers, 31 parts, among them J1 USB_B_Micro, J2 Conn_01x26, J3 Conn_01x26, SW1 Prog, U1 LP38691SD-3.3, U2 MKL02Z32VFG4, U3 MK20DX256VLH7, Y1 32.768 KHz, Y2 16 MHz

Commit message: fin pcb
Routing:
- net GND: track 67.6 -> 68.8 mm, vias 8 -> 9
Other:
- board outline added: 69 x 34 mm
- board text added: "Hecho en Argentina"
- board text added: "Teensy 3.2 clone"
Changed lines of the file:
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@@
   (general
     (thickness 1.6)
-    (drawings 1)
-    (tracks 527)
+    (drawings 9)
+    (tracks 530)
     (zones 0)
     (modules 31)
@@
     (aux_axis_origin 12 12)
     (grid_origin 12 12)
-    (visible_elements FFFFFF7F)
+    (visible_elements FFFDFF7F)
     (pcbplotparams
       (layerselection 0x010fc_ffffffff)
@@
     (tags "QFN NoLead")
     (attr smd)
-    (fp_text reference U2 (at 3.25 1.25) (layer F.SilkS)
+    (fp_text reference U2 (at 1.25 3) (layer F.SilkS)
       (effects (font (size 1 1) (thickness 0.15)))
     )
@@
     (descr "Through hole straight socket strip, 1x26, 2.54mm pitch, single row (from Kicad 4.0.7), script generated")
     (tags "Through hole socket strip THT 1x26 2.54mm single row")
-    (fp_text reference J3 (at 0 -2.77 90) (layer F.SilkS)
+    (fp_text reference J3 (at 2.5 -1 180) (layer F.SilkS)
       (effects (font (size 1 1) (thickness 0.15)))
     )
@@
     (descr "Through hole straight socket strip, 1x26, 2.54mm pitch, single row (from Kicad 4.0.7), script generated")
     (tags "Through hole socket strip THT 1x26 2.54mm single row")
-    (fp_text reference J2 (at 0 -2.77 90) (layer F.SilkS)
+    (fp_text reference J2 (at -2.5 -0.5 180) (layer F.SilkS)
       (effects (font (size 1 1) (thickness 0.15)))
     )
@@
     (tags "SMD SMT crystal")
     (attr smd)
-    (fp_text reference Y2 (at 0 -2) (layer F.SilkS)
+    (fp_text reference Y2 (at 0 2) (layer F.SilkS)
       (effects (font (size 1 1) (thickness 0.15)))
     )
@@
     (tags "SMD SMT crystal")
     (attr smd)
-    (fp_text reference Y1 (at 0 -1.8 90) (layer F.SilkS)
+    (fp_text reference Y1 (at -2 -0.25 180) (layer F.SilkS)
       (effects (font (size 1 1) (thickness 0.15)))
     )
@@
     (tags resistor)
     (attr smd)
-    (fp_text reference R4 (at 0 -1.65) (layer F.SilkS)
+    (fp_text reference R4 (at -3.0625 0.5) (layer F.SilkS)
       (effects (font (size 1 1) (thickness 0.15)))
     )
@@
     (tags resistor)
     (attr smd)
-    (fp_text reference R3 (at 0 -1.65) (layer F.SilkS)
+    (fp_text reference R3 (at 0 1.5) (layer F.SilkS)
       (effects (font (size 1 1) (thickness 0.15)))
     )
@@
     (tags resistor)
     (attr smd)
-    (fp_text reference R2 (at 0 -1.65) (layer F.SilkS)
+    (fp_text reference R2 (at -3 -0.5) (layer F.SilkS)
       (effects (font (size 1 1) (thickness 0.15)))
     )
@@
     (tags resistor)
     (attr smd)
-    (fp_text reference R1 (at 0 -1.65) (layer F.SilkS)
+    (fp_text reference R1 (at -3 0) (layer F.SilkS)
       (effects (font (size 1 1) (thickness 0.15)))
     )
@@
     (tags capacitor)
     (attr smd)
-    (fp_text reference C10 (at 0 -1.65) (layer F.SilkS)
+    (fp_text reference C10 (at 0 1.5) (layer F.SilkS)
       (effects (font (size 1 1) (thickness 0.15)))
     )
@@
     (tags capacitor)
     (attr smd)
-    (fp_text reference C6 (at 0 -1.65) (layer F.SilkS)
+    (fp_text reference C6 (at -0.5625 2) (layer F.SilkS)
       (effects (font (size 1 1) (thickness 0.15)))
     )
@@
     (tags capacitor)
     (attr smd)
-    (fp_text reference C5 (at 0 -1.65 90) (layer F.SilkS)
+    (fp_text reference C5 (at 0.0625 2 180) (layer F.SilkS)
       (effects (font (size 1 1) (thickness 0.15)))
     )
@@
     (tags capacitor)
     (attr smd)
-    (fp_text reference C1 (at 0 -1.65 90) (layer F.SilkS)
+    (fp_text reference C1 (at 0 2 180) (layer F.SilkS)
       (effects (font (size 1 1) (thickness 0.15)))
     )
@@
     (tags capacitor)
     (attr smd)
-    (fp_text reference C2 (at 0 -1.65) (layer F.SilkS)
+    (fp_text reference C2 (at 0 1.5) (layer F.SilkS)
       (effects (font (size 1 1) (thickness 0.15)))
     )
@@
     (tags capacitor)
     (attr smd)
-    (fp_text reference C3 (at -0.0625 2 90) (layer F.SilkS)
+    (fp_text reference C3 (at -2.5 0.5 180) (layer F.SilkS)
       (effects (font (size 1 1) (thickness 0.15)))
     )
@@
     (tags capacitor)
     (attr smd)
-    (fp_text reference C4 (at 0 -1.65 90) (layer F.SilkS)
+    (fp_text reference C4 (at 0.5 -2 180) (layer F.SilkS)
       (effects (font (size 1 1) (thickness 0.15)))
     )
@@
     (tags capacitor)
     (attr smd)
-    (fp_text reference C8 (at 0 -1.65 90) (layer F.SilkS)
+    (fp_text reference C8 (at -2.5625 0 180) (layer F.SilkS)
       (effects (font (size 1 1) (thickness 0.15)))
     )
@@
     (tags capacitor)
     (attr smd)
-    (fp_text reference C9 (at 0 -1.65) (layer F.SilkS)
+    (fp_text reference C9 (at 0.0625 -1.5) (layer F.SilkS)
       (effects (font (size 1 1) (thickness 0.15)))
     )
@@
     (tags "huson nolead SOT1061")
     (attr smd)
-    (fp_text reference D1 (at -2.5 0) (layer F.SilkS)
+    (fp_text reference D1 (at -2.5 0.5) (layer F.SilkS)
       (effects (font (size 1 1) (thickness 0.15)))
     )
@@
     (tags diode)
     (attr smd)
-    (fp_text reference D2 (at 0 -1.65) (layer F.SilkS)
+    (fp_text reference D2 (at 3.0625 0.5) (layer F.SilkS)
       (effects (font (size 1 1) (thickness 0.15)))
     )
@@
     (tags resistor)
     (attr smd)
-    (fp_text reference F1 (at 0 -1.65) (layer F.SilkS)
+    (fp_text reference F1 (at -1.4375 -2) (layer F.SilkS)
       (effects (font (size 1 1) (thickness 0.15)))
     )
@@
     (tags "solder jumper open")
     (attr virtual)
-    (fp_text reference JP1 (at 0 -1.8) (layer F.SilkS)
+    (fp_text reference JP1 (at -0.85 2) (layer F.SilkS)
       (effects (font (size 1 1) (thickness 0.15)))
     )
@@
     (tags "SPST Button Switch")
     (attr smd)
-    (fp_text reference SW1 (at 0 -2.6) (layer F.SilkS)
+    (fp_text reference SW1 (at 0 2.5) (layer F.SilkS)
       (effects (font (size 1 1) (thickness 0.15)))
     )
@@
     (tags "WSON6 0.95")
     (attr smd)
-    (fp_text reference U1 (at 0 -2.575 90) (layer F.SilkS)
+    (fp_text reference U1 (at -3 -1 180) (layer F.SilkS)
       (effects (font (size 1 1) (thickness 0.15)))
     )
@@
     (tags "LQFP QFP")
     (attr smd)
-    (fp_text reference U3 (at 0 -7.4 135) (layer F.SilkS)
+    (fp_text reference U3 (at 1.767767 -7.424621 315) (layer F.SilkS)
       (effects (font (size 1 1) (thickness 0.15)))
     )
@@
     )
   )
+  (dimension 34 (width 0.15) (layer Dwgs.User)
+    (gr_text "34.000 mm" (at 173.3 94 90) (layer Dwgs.User)
+      (effects (font (size 1 1) (thickness 0.15)))
+    )
+    (feature1 (pts (xy 169 77) (xy 172.586421 77)))
+    (feature2 (pts (xy 169 111) (xy 172.586421 111)))
+    (crossbar (pts (xy 172 111) (xy 172 77)))
+    (arrow1a (pts (xy 172 77) (xy 172.586421 78.126504)))
+    (arrow1b (pts (xy 172 77) (xy 171.413579 78.126504)))
+    (arrow2a (pts (xy 172 111) (xy 172.586421 109.873496)))
+    (arrow2b (pts (xy 172 111) (xy 171.413579 109.873496)))
+  )
+  (dimension 69 (width 0.15) (layer Dwgs.User)
+    (gr_text "69.000 mm" (at 134.5 73.2) (layer Dwgs.User)
+      (effects (font (size 1 1) (thickness 0.15)))
+    )
+    (feature1 (pts (xy 169 77) (xy 169 73.913579)))
+    (feature2 (pts (xy 100 77) (xy 100 73.913579)))
+    (crossbar (pts (xy 100 74.5) (xy 169 74.5)))
+    (arrow1a (pts (xy 169 74.5) (xy 167.873496 75.086421)))
+    (arrow1b (pts (xy 169 74.5) (xy 167.873496 73.913579)))
+    (arrow2a (pts (xy 100 74.5) (xy 101.126504 75.086421)))
+    (arrow2b (pts (xy 100 74.5) (xy 101.126504 73.913579)))
+  )
+  (gr_text "Hecho en Argentina" (at 167.5 105) (layer F.SilkS)
+    (effects (font (size 1 1) (thickness 0.15)) (justify right))
+  )
+  (gr_text "Teensy 3.2 clone" (at 167.5 103) (layer F.SilkS)
+    (effects (font (size 1 1) (thickness 0.2)) (justify right))
+  )
+  (gr_line (start 100 111) (end 100 77) (layer Edge.Cuts) (width 0.05))
+  (gr_line (start 169 111) (end 100 111) (layer Edge.Cuts) (width 0.05))
+  (gr_line (start 169 77) (end 169 111) (layer Edge.Cuts) (width 0.05))
+  (gr_line (start 100 77) (end 169 77) (layer Edge.Cuts) (width 0.05))
   (gr_text "Mínimos (Mayer 8 mils):\nGrillas: 0. 5mm, 0.25 mm\nVía: 0.8 mm (0.4 mm)\nMargen: 0.18 mm\nPista: 0.20 mm\nDist. a borde: 0.30 mm\nTerminación: HASL" (at 182.25 93.25) (layer Dwgs.User)
     (effects (font (size 1 1) (thickness 0.15)) (justify left))
@@
   (segment (start 146 102.5) (end 147 103.5) (width 0.2) (layer F.Cu) (net 1))
   (segment (start 145.5 102.5) (end 146 102.5) (width 0.2) (layer F.Cu) (net 1))
+  (via (at 108.25 104.5) (size 0.8) (drill 0.4) (layers F.Cu B.Cu) (net 1))
+  (segment (start 108 104.25) (end 108.25 104.5) (width 0.2) (layer F.Cu) (net 1))
+  (segment (start 108 103.34) (end 108 104.25) (width 0.2) (layer F.Cu) (net 1))
   (segment (start 103.319999 86.680001) (end 104 86) (width 0.2) (layer F.Cu) (net 2))
   (segment (start 103.319999 91.449001) (end 103.319999 86.680001) (width 0.2) (layer F.Cu) (net 2))

Commit message: ajustes
Parts:
- added FID2: Fiducial, Fiducial:Fiducial_0.5mm_Mask1.5mm, F.Cu at (157.5, 83.0)
- added FID3: Fiducial, Fiducial:Fiducial_0.5mm_Mask1.5mm, F.Cu at (118.0, 104.5)
Routing:
- net /AGND: track 44.0 -> 42.6 mm
- net /AREF: track 40.9 -> 40.2 mm

Commit message: ajustes revision pcb
Parts:
- moved FID1 3.00 mm to (166.0, 96.5)
Connections:
- net /AGND renamed GNDA
Routing:
- net Net-(J3-Pad18): track 15.9 -> 14.7 mm
- net Net-(J3-Pad17): track 16.8 -> 15.8 mm
Other:
- board text added: "+"
- board text added: "-"
- board text added: "v1.0 - 06/2020"
